Commit message: addmid

File: limo_description/urdf/limo_four_diff.xacro (robot description, xacro)
@@ -17,4 +17,66 @@
         <origin xyz="0.0 0.0 -0.15" rpy="0 0 0"/>
     </joint>
+    <!-- === Livox Mid360 Lidar === -->
+  <joint name="mid360_joint" type="fixed">
+    <parent link="base_link"/>
+    <!-- 位于原雷达位置：前方略微上方 -->
+    <child link="mid360_link"/>
+    <origin xyz="0.0 0 0.122" rpy="0 0 0"/>
+  </joint>
+  <link name="mid360_link">
+    <visual>
+      <origin xyz="0 0 0" rpy="0 0 0"/>
+      <geometry>
+        <!-- 可自行换成实际 mesh 模型 -->
+        <cylinder length="0.05" radius="0.04"/>
+      </geometry>
+      <material name="gray"/>
+    </visual>
+  </link>
+  <gazebo reference="mid360_link">
+    <sensor type="ray" name="laser_livox">
+            <pose>0 0 0.0 0 0 0</pose>
+            <visualize>true</visualize>
+            <always_on>true</always_on>
+            <update_rate>20</update_rate>
+            <!-- This ray plgin is only for visualization. -->
+            <plugin name="gazebo_ros_laser_controller" filename="liblivox_laser_simulation.so">
+            <ray>
+            <scan>
+              <horizontal>
+                <samples>100</samples>
+                <resolution>1</resolution>
+                <min_angle>-3.1415926535897931</min_angle>
+                <max_angle>3.1415926535897931</max_angle>
+              </horizontal>
+              <vertical>
+                <samples>50</samples>
+                <resolution>1</resolution>
+                <min_angle>-3.1415926535897931</min_angle>
+                <max_angle>3.1415926535897931</max_angle>
+              </vertical>
+            </scan>
+            <range>
+              <min>0.1</min>
+              <max>40</max>
+              <resolution>1</resolution>
+            </range>
+            <noise>
+              <type>gaussian</type>
+              <mean>0.0</mean>
+              <stddev>0.0</stddev>
+            </noise>
+            </ray>
+              <visualize>false</visualize>
+              <samples>20000</samples>
+              <downsample>1</downsample>
+              <csv_file_name>mid360-real-centr.csv</csv_file_name>
+              <publish_pointcloud_type>2</publish_pointcloud_type>
+              <ros_topic>/livox/lidar</ros_topic>
+              <frameName>mid360_link</frameName>
+            </plugin>
+        </sensor>
+      <!-- === End Mid360 === -->
+    </gazebo>
     <!-- Base link -->
     <link name="base_link">

Commit message: retation

File: limo_description/urdf/limo_four_diff.xacro (robot description, xacro)
@@ -22,5 +22,5 @@
     <!-- 位于原雷达位置：前方略微上方 -->
     <child link="mid360_link"/>
-    <origin xyz="0.0 0 0.122" rpy="0 0 0"/>
+    <origin xyz="0.0 0 0.122" rpy="0 0 -1.57"/>
   </joint>
   <link name="mid360_link">

Commit message: addmid

File: limo_description/urdf/limo_four_diff.xacro (robot description, xacro)
@@ -11,4 +11,7 @@
     <xacro:property name="wheel_length" value="0.0437" />
     <xacro:property name="wheel_radius" value="0.048" />
+    <material name="gray">
+    <color rgba="0.5 0.5 0.5 1"/>
+    </material>
     <link name="base_footprint"/>
     <joint name="base_joint" type="fixed">

Commit message: end

File: limo_description/urdf/limo_four_diff.xacro (robot description, xacro)
@@ -25,5 +25,5 @@
     <!-- 位于原雷达位置：前方略微上方 -->
     <child link="mid360_link"/>
-    <origin xyz="0.0 0 0.122" rpy="0 0 -1.57"/>
+    <origin xyz="0.0 0 0.122" rpy="0 0 -1.6"/>
   </joint>
   <link name="mid360_link">

Commit message: fix

File: limo_description/urdf/limo_four_diff.xacro (robot description, xacro)
@@ -25,5 +25,5 @@
     <!-- 位于原雷达位置：前方略微上方 -->
     <child link="mid360_link"/>
-    <origin xyz="0.0 0 0.122" rpy="0 0 -1.6"/>
+    <origin xyz="0.0 0 0.122" rpy="0 0 -1.62"/>
   </joint>
   <link name="mid360_link">

Commit message: new

File: limo_description/urdf/limo_four_diff.xacro (robot description, xacro)
@@ -104,7 +104,7 @@
         </inertial>
     </link>
-    <!-- <xacro:limo_laser parent_prefix="base_link" frame_prefix="laser">
+    <xacro:limo_laser parent_prefix="base_link" frame_prefix="laser">
         <origin xyz="0.103 0 -0.034" rpy="0 0 0"/>
-    </xacro:limo_laser> -->
+    </xacro:limo_laser>
     <xacro:limo_depth_camera parent_prefix="base_link" frame_prefix="depth_camera">
         <origin xyz="0.084 0 0.03" rpy="0 0 0"/>
@@ -125,3 +125,63 @@
         <origin xyz="${-wheelbase/2} ${-track/2} ${wheel_vertical_offset}" rpy="${M_PI} 0 0" />
     </xacro:limo_wheel>
+    <gazebo reference="base_link">
+    <sensor name='collision_sensor' type='contact'>
+      <contact>
+        <collision>base_link_collision</collision>
+      </contact>
+      <plugin name="collision_sensor" filename="libgazebo_collision_sensor.so">
+        <rosDebugLevel>na</rosDebugLevel>
+        <topicName>/gazebo/base_collision</topicName>
+        <updateRate>20.0</updateRate>
+      </plugin>
+    </sensor>
+  </gazebo>
+  <gazebo reference="front_left_wheel_link">
+  <sensor name="fl_collision_sensor" type="contact">
+    <contact>
+      <collision>front_left_wheel_link_collision</collision>
+    </contact>
+    <plugin name="fl_collision_plugin"
+            filename="libgazebo_collision_sensor.so">
+      <topicName>/gazebo/front_left_collision</topicName>
+      <updateRate>20.0</updateRate>
+    </plugin>
+  </sensor>
+</gazebo>
+<gazebo reference="front_right_wheel_link">
+  <sensor name="fr_collision_sensor" type="contact">
+    <contact>
+      <collision>front_right_wheel_link_collision</collision>
+    </contact>
+    <plugin name="fr_collision_plugin"
+            filename="libgazebo_collision_sensor.so">
+      <topicName>/gazebo/front_right_collision</topicName>
+      <updateRate>20.0</updateRate>
+    </plugin>
+  </sensor>
+</gazebo>
+<gazebo reference="rear_left_wheel_link">
+  <sensor name="rl_collision_sensor" type="contact">
+    <contact>
+      <collision>rear_left_wheel_link_collision</collision>
+    </contact>
+    <plugin name="rl_collision_plugin"
+            filename="libgazebo_collision_sensor.so">
+      <topicName>/gazebo/rear_left_collision</topicName>
+      <updateRate>20.0</updateRate>
+    </plugin>
+  </sensor>
+</gazebo>
+<gazebo reference="rear_right_wheel_link">
+  <sensor name="rr_collision_sensor" type="contact">
+    <contact>
+      <collision>rear_right_wheel_link_collision</collision>
+    </contact>
+    <plugin name="rr_collision_plugin"
+            filename="libgazebo_collision_sensor.so">
+      <topicName>/gazebo/rear_right_collision</topicName>
+      <updateRate>20.0</updateRate>
+    </plugin>
+  </sensor>
+</gazebo>
 </robot>

Commit message: add new

File: limo_description/urdf/limo_four_diff.xacro (robot description, xacro)
@@ -104,4 +104,14 @@
         </inertial>
     </link>
+    <link name="safety_collision_link"> <!-- collision -->
+    <collision name="safety_collision">
+    <origin xyz="0 0 -0.05" rpy="0 0 0"/>
+    <geometry> <cylinder radius="0.18" length="0.10"/> </geometry>
+    </collision> <!-- visual -->
+    <visual name="safety_visual"> <origin xyz="0 0 -0.05" rpy="0 0 0"/> <geometry>
+    <cylinder radius="0.18" length="0.10"/> </geometry>
+     <material name="transparent_red"/> </visual> <!-- inertia --> <inertial> <origin xyz="0 0 0"/> <mass value="0.001"/> <inertia ixx="1e-6" ixy="0" ixz="0" iyy="1e-6" iyz="0" izz="1e-6"/> </inertial> </link>
+    <!-- fixed joint -->
+    <joint name="safety_collision_joint" type="fixed"> <parent link="base_link"/> <child link="safety_collision_link"/> <origin xyz="0 0 0" rpy="0 0 0"/> </joint>
     <xacro:limo_laser parent_prefix="base_link" frame_prefix="laser">
         <origin xyz="0.103 0 -0.034" rpy="0 0 0"/>
@@ -125,5 +135,5 @@
         <origin xyz="${-wheelbase/2} ${-track/2} ${wheel_vertical_offset}" rpy="${M_PI} 0 0" />
     </xacro:limo_wheel>
-    <gazebo reference="base_link">
+    <!-- <gazebo reference="base_link">
     <sensor name='collision_sensor' type='contact'>
       <contact>
@@ -136,52 +146,16 @@
       </plugin>
     </sensor>
+  </gazebo> -->
+      <gazebo reference="safety_collision_link">
+    <sensor name='collision_sensor' type='contact'>
+      <contact>
+        <collision>base_link_fixed_joint_lump__safety_collision_collision_1</collision>
+      </contact>
+      <plugin name="collision_sensor" filename="libgazebo_collision_sensor.so">
+        <rosDebugLevel>na</rosDebugLevel>
+        <topicName>/gazebo/base_collision</topicName>
+        <updateRate>20.0</updateRate>
+      </plugin>
+    </sensor>
   </gazebo>
-  <gazebo reference="front_left_wheel_link">
-  <sensor name="fl_collision_sensor" type="contact">
-    <contact>
-      <collision>front_left_wheel_link_collision</collision>
-    </contact>
-    <plugin name="fl_collision_plugin"
-            filename="libgazebo_collision_sensor.so">
-      <topicName>/gazebo/front_left_collision</topicName>
-      <updateRate>20.0</updateRate>
-    </plugin>
-  </sensor>
-</gazebo>
-<gazebo reference="front_right_wheel_link">
-  <sensor name="fr_collision_sensor" type="contact">
-    <contact>
-      <collision>front_right_wheel_link_collision</collision>
-    </contact>
-    <plugin name="fr_collision_plugin"
-            filename="libgazebo_collision_sensor.so">
-      <topicName>/gazebo/front_right_collision</topicName>
-      <updateRate>20.0</updateRate>
-    </plugin>
-  </sensor>
-</gazebo>
-<gazebo reference="rear_left_wheel_link">
-  <sensor name="rl_collision_sensor" type="contact">
-    <contact>
-      <collision>rear_left_wheel_link_collision</collision>
-    </contact>
-    <plugin name="rl_collision_plugin"
-            filename="libgazebo_collision_sensor.so">
-      <topicName>/gazebo/rear_left_collision</topicName>
-      <updateRate>20.0</updateRate>
-    </plugin>
-  </sensor>
-</gazebo>
-<gazebo reference="rear_right_wheel_link">
-  <sensor name="rr_collision_sensor" type="contact">
-    <contact>
-      <collision>rear_right_wheel_link_collision</collision>
-    </contact>
-    <plugin name="rr_collision_plugin"
-            filename="libgazebo_collision_sensor.so">
-      <topicName>/gazebo/rear_right_collision</topicName>
-      <updateRate>20.0</updateRate>
-    </plugin>
-  </sensor>
-</gazebo>
 </robot>
