Commit message: change

File: limo_description/urdf/limo_four_diff.xacro (robot description, xacro)
@@ -104,14 +104,6 @@
         </inertial>
     </link>
-    <link name="safety_collision_link"> <!-- collision -->
-    <collision name="safety_collision">
-    <origin xyz="0 0 -0.05" rpy="0 0 0"/>
-    <geometry> <cylinder radius="0.18" length="0.10"/> </geometry>
-    </collision> <!-- visual -->
-    <visual name="safety_visual"> <origin xyz="0 0 -0.05" rpy="0 0 0"/> <geometry>
-    <cylinder radius="0.18" length="0.10"/> </geometry>
-     <material name="transparent_red"/> </visual> <!-- inertia --> <inertial> <origin xyz="0 0 0"/> <mass value="0.001"/> <inertia ixx="1e-6" ixy="0" ixz="0" iyy="1e-6" iyz="0" izz="1e-6"/> </inertial> </link>
     <!-- fixed joint -->
-    <joint name="safety_collision_joint" type="fixed"> <parent link="base_link"/> <child link="safety_collision_link"/> <origin xyz="0 0 0" rpy="0 0 0"/> </joint>
+    <!-- <joint name="safety_collision_joint" type="fixed"> <parent link="base_link"/> <child link="safety_collision_link"/> <origin xyz="0 0 0" rpy="0 0 0"/> </joint> -->
     <xacro:limo_laser parent_prefix="base_link" frame_prefix="laser">
         <origin xyz="0.103 0 -0.034" rpy="0 0 0"/>
@@ -135,5 +127,5 @@
         <origin xyz="${-wheelbase/2} ${-track/2} ${wheel_vertical_offset}" rpy="${M_PI} 0 0" />
     </xacro:limo_wheel>
-    <!-- <gazebo reference="base_link">
+    <gazebo reference="base_link">
     <sensor name='collision_sensor' type='contact'>
       <contact>
@@ -146,6 +138,6 @@
       </plugin>
     </sensor>
-  </gazebo> -->
-      <gazebo reference="safety_collision_link">
+  </gazebo>
+      <!-- <gazebo reference="safety_collision_link">
     <sensor name='collision_sensor' type='contact'>
       <contact>
@@ -158,4 +150,4 @@
       </plugin>
     </sensor>
-  </gazebo>
+  </gazebo> -->
 </robot>

File: limo_description/urdf/limo_xacro.xacro (robot description, xacro)
@@ -26,4 +26,6 @@
             <xacro:insert_block name="joint_pose"/>
             <axis xyz="0 ${reflect*1} 0"/>
+            <dynamics damping="0.01" friction="0.0"/>
+            <limit effort="1.1" velocity="24"/>
         </joint>
     </xacro:macro>

Commit message: add tf and change tf

File: limo_description/urdf/limo_four_diff.xacro (robot description, xacro)
@@ -15,4 +15,12 @@
     </material>
     <link name="base_footprint"/>
+    <!-- Rear axle center coordinate frame -->
+    <link name="rear_axle_link"/>
+    <joint name="rear_axle_joint" type="fixed">
+        <parent link="base_link"/>
+        <child link="rear_axle_link"/>
+        <origin xyz="${-wheelbase/2} 0 ${wheel_vertical_offset}"
+                rpy="0 0 0"/>
+    </joint>
     <joint name="base_joint" type="fixed">
         <parent link="base_link"/>
@@ -153,11 +161,11 @@
   <!-- Front Left Wheel: Zero Contact Friction -->
   <gazebo reference="front_left_wheel_link">
-      <mu1>0.05</mu1>
-      <mu2>0.05</mu2>
+      <mu1>0.1</mu1>
+      <mu2>0.1</mu2>
   </gazebo>
   <!-- Front Right Wheel: Zero Contact Friction -->
   <gazebo reference="front_right_wheel_link">
-      <mu1>0.05</mu1>
-      <mu2>0.05</mu2>
+      <mu1>0.1</mu1>
+      <mu2>0.1</mu2>
   </gazebo>
   <!-- Rear Left Wheel: Increased Contact Friction -->
