Commit message: chang damping

File: limo_description/urdf/limo_xacro.xacro (robot description, xacro)
@@ -26,5 +26,5 @@
             <xacro:insert_block name="joint_pose"/>
             <axis xyz="0 ${reflect*1} 0"/>
-            <dynamics damping="0.01" friction="0.0"/>
+            <dynamics damping="0.0" friction="0.0"/>
             <limit effort="1.1" velocity="24"/>
         </joint>
